File: pcb/OpenPDCharger.sch (KiCad schematic (older format))
At the start: 0 parts

Commit message: update
Changed lines of the file:
@@
 $Descr A4 11693 8268
 encoding utf-8
-Sheet 1 9
+Sheet 1 10
 Title ""
 Date ""
@@
 F0 "MCU" 50
 F1 "mcu.sch" 50
+F2 "USBPDFS_D_N" I L -1950 3600 50
+F3 "USBPDFS_D_P" I L -1950 3500 50
+F4 "USBPD_CC2" I L -1950 3800 50
+F5 "USBPD_CC1" I L -1950 3700 50
 $EndSheet
 $Sheet
-S -400 2300 1100 850
+S -1900 1550 1100 850
 U 5E5B0438
 F0 "POWER" 50
 F1 "power.sch" 50
+F2 "USBPD_1A_PROTECT" I L -1900 1800 50
+F3 "USBPD_550mA_PROTECT" I L -1900 1700 50
 $EndSheet
 $Sheet
@@
 F1 "usb.sch" 50
 F2 "USB_DM" I L 1800 1650 50
+F3 "USB_DP" I L 1800 1550 50
 $EndSheet
 $Sheet
@@
 Wire Wire Line
 	4150 5350 4050 5350
+$Sheet
+S 8500 4900 1150 1050
+U 5E6679B9
+F0 "NiMH Charger" 50
+F1 "nihm_charger.sch" 50
+F2 "NIHM_ENABLE" I L 8500 5000 50
+F3 "~NIHM_TOC" I L 8500 5150 50
+F4 "~NIHM_FAULT" I L 8500 5250 50
+F5 "~NIHM_CHRG" I L 8500 5350 50
+F6 "~NIHM_RDY" I L 8500 5450 50
+$EndSheet
 $EndSCHEMATC
