File: pcb/battery_management.sch (KiCad schematic (older format))
At the start: 19 parts, among them Q10 CSD17573Q5B, Q8 CSD17573Q5B, Q9 FDN358P, U8 BQ4050RSMR

Commit message: update
Parts:
- added C57: 100nF, symbol Device:C
- added R52, R54: 100, symbol Device:R
- added R53: 0.01, symbol Device:R
- added R55, R56, R57, R58: 10K, symbol Device:R
- Q9: footprint SSOT-3 -> Lib:SSOT-3
Connections:
- net GND: now also R53.1, R54.2; no longer U8.33 (EP), U8.33_1 (EP), U8.9 (VSS)
- net at U8.10 (TS1): now also R55.1
- net at U8.11 (TS2): now also R56.1
- net at U8.12 (TS3): now also R57.1
- net at U8.13 (TS4): now also R58.1
- net BAT_GND: now reaches U8.25 (FUSE)
- net BAT_GND: now also U8.33 (EP), U8.33_1 (EP), U8.9 (VSS), R52.2, R53.2, R55.2, R56.2, R57.2, R58.2
- net at U8.6 (SRN): now also C57.2, R54.1
- net at U8.8 (SRP): now also C57.1, R52.1
Changed lines of the file:
@@
 $Descr A4 11693 8268
 encoding utf-8
-Sheet 9 9
+Sheet 9 10
 Title ""
 Date ""
@@
 	1    0    0    -1
 $EndComp
-$Comp
-L power:GND #PWR0145
-U 1 1 5E5FADD6
-P 5500 6850
-F 0 "#PWR0145" H 5500 6600 50  0001 C CNN
-F 1 "GND" H 5505 6677 50  0000 C CNN
-F 2 "" H 5500 6850 50  0001 C CNN
-F 3 "" H 5500 6850 50  0001 C CNN
-	1    5500 6850
-	1    0    0    -1
-$EndComp
 Wire Wire Line
 	5450 6800 5500 6800
@@
 F 0 "Q9" V 6735 2500 50  0000 C CNN
 F 1 "FDN358P" V 6644 2500 50  0000 C CNN
-F 2 "SSOT-3" H 6500 2500 50  0001 L BNN
+F 2 "Lib:SSOT-3" H 6500 2500 50  0001 L BNN
 F 3 "" H 6500 2500 50  0001 C CNN
 	1    6500 2500
@@
 Wire Wire Line
 	3800 3100 5900 3100
-Wire Wire Line
-	3800 3100 2750 3100
-Connection ~ 3800 3100
 $Comp
 L Device:R R37
@@
 	3200 5200 3850 5200
 Connection ~ 3200 5000
+Wire Wire Line
+	5450 5300 5500 5300
+Wire Wire Line
+	5500 5300 5500 5350
+$Comp
+L Device:R R53
+U 1 1 5E6B7480
+P 2550 3450
+F 0 "R53" V 2343 3450 50  0000 C CNN
+F 1 "0.01" V 2434 3450 50  0000 C CNN
+F 2 "" V 2480 3450 50  0001 C CNN
+F 3 "~" H 2550 3450 50  0001 C CNN
+	1    2550 3450
+	0    1    1    0
+$EndComp
+$Comp
+L Device:R R52
+U 1 1 5E6B7B24
+P 2350 3700
+F 0 "R52" H 2280 3654 50  0000 R CNN
+F 1 "100" H 2280 3745 50  0000 R CNN
+F 2 "" V 2280 3700 50  0001 C CNN
+F 3 "~" H 2350 3700 50  0001 C CNN
+	1    2350 3700
+	-1   0    0    1
+$EndComp
+$Comp
+L Device:R R54
+U 1 1 5E6B898E
+P 2750 3700
+F 0 "R54" H 2680 3654 50  0000 R CNN
+F 1 "100" H 2680 3745 50  0000 R CNN
+F 2 "" V 2680 3700 50  0001 C CNN
+F 3 "~" H 2750 3700 50  0001 C CNN
+	1    2750 3700
+	-1   0    0    1
+$EndComp
+$Comp
+L Device:C C57
+U 1 1 5E6B8C9C
+P 2550 4200
+F 0 "C57" V 2802 4200 50  0000 C CNN
+F 1 "100nF" V 2711 4200 50  0000 C CNN
+F 2 "" H 2588 4050 50  0001 C CNN
+F 3 "~" H 2550 4200 50  0001 C CNN
+	1    2550 4200
+	0    -1   -1   0
+$EndComp
+Wire Wire Line
+	2700 4200 2750 4200
+Wire Wire Line
+	2750 4200 2750 3850
+Wire Wire Line
+	2700 3450 2750 3450
+Wire Wire Line
+	2750 3450 2750 3550
+Wire Wire Line
+	2350 3550 2350 3450
+Wire Wire Line
+	2350 3450 2400 3450
+Wire Wire Line
+	2400 4200 2350 4200
+Wire Wire Line
+	2350 4200 2350 3850
+Connection ~ 2750 4200
+Wire Wire Line
+	3850 5500 2350 5500
+Connection ~ 2350 4200
+$Comp
+L Device:R R55
+U 1 1 5E6D9142
+P 3550 5700
+F 0 "R55" V 3500 5450 50  0000 C CNN
+F 1 "10K" V 3500 5900 50  0000 C CNN
+F 2 "" V 3480 5700 50  0001 C CNN
+F 3 "~" H 3550 5700 50  0001 C CNN
+	1    3550 5700
+	0    1    1    0
+$EndComp
+Wire Wire Line
+	3850 5700 3700 5700
+$Comp
+L Device:R R56
+U 1 1 5E6DD663
+P 3550 5800
+F 0 "R56" V 3500 5550 50  0000 C CNN
+F 1 "10K" V 3500 6000 50  0000 C CNN
+F 2 "" V 3480 5800 50  0001 C CNN
+F 3 "~" H 3550 5800 50  0001 C CNN
+	1    3550 5800
+	0    1    1    0
+$EndComp
+Wire Wire Line
+	3850 5800 3700 5800
+$Comp
+L Device:R R57
+U 1 1 5E6DFA6F
+P 3550 5900
+F 0 "R57" V 3500 5650 50  0000 C CNN
+F 1 "10K" V 3500 6100 50  0000 C CNN
+F 2 "" V 3480 5900 50  0001 C CNN
+F 3 "~" H 3550 5900 50  0001 C CNN
+	1    3550 5900
+	0    1    1    0
+$EndComp
+Wire Wire Line
+	3850 5900 3700 5900
+$Comp
+L Device:R R58
+U 1 1 5E6E1E48
+P 3550 6000
+F 0 "R58" V 3500 5750 50  0000 C CNN
+F 1 "10K" V 3500 6200 50  0000 C CNN
+F 2 "" V 3480 6000 50  0001 C CNN
+F 3 "~" H 3550 6000 50  0001 C CNN
+	1    3550 6000
+	0    1    1    0
+$EndComp
+Wire Wire Line
+	3850 6000 3700 6000
+Wire Wire Line
+	3400 6000 3150 6000
+Wire Wire Line
+	3150 5900 3400 5900
+Wire Wire Line
+	3400 5800 3150 5800
+Wire Wire Line
+	3150 5700 3400 5700
+Wire Wire Line
+	3150 6050 3150 6000
+Wire Wire Line
+	3150 5900 3150 5800
+Wire Wire Line
+	3150 6000 3150 5900
+Connection ~ 3150 6000
+Connection ~ 3150 5900
+Wire Wire Line
+	3150 5800 3150 5700
+Connection ~ 3150 5800
+$Comp
+L openpcharger:BAT_GND #PWR0170
+U 1 1 5E6FE22F
+P 3150 6050
+F 0 "#PWR0170" H 2850 5800 50  0001 C CNN
+F 1 "BAT_GND" H 3155 5877 50  0000 C CNN
+F 2 "" H 3150 6050 50  0001 C CNN
+F 3 "" H 3150 6050 50  0001 C CNN
+	1    3150 6050
+	1    0    0    -1
+$EndComp
+$Comp
+L openpcharger:BAT_GND #PWR0171
+U 1 1 5E6FEE1E
+P 5500 6850
+F 0 "#PWR0171" H 5200 6600 50  0001 C CNN
+F 1 "BAT_GND" H 5505 6677 50  0000 C CNN
+F 2 "" H 5500 6850 50  0001 C CNN
+F 3 "" H 5500 6850 50  0001 C CNN
+	1    5500 6850
+	1    0    0    -1
+$EndComp
+$Comp
+L openpcharger:BAT_GND #PWR0172
+U 1 1 5E6FF2D1
+P 5500 5350
+F 0 "#PWR0172" H 5200 5100 50  0001 C CNN
+F 1 "BAT_GND" H 5505 5177 50  0000 C CNN
+F 2 "" H 5500 5350 50  0001 C CNN
+F 3 "" H 5500 5350 50  0001 C CNN
+	1    5500 5350
+	1    0    0    -1
+$EndComp
+Wire Wire Line
+	2750 4200 2750 5400
+Wire Wire Line
+	2750 5400 3850 5400
+Wire Wire Line
+	2350 4200 2350 5500
+Wire Wire Line
+	2350 3450 2050 3450
+Connection ~ 2350 3450
+Wire Wire Line
+	2050 3550 2050 3450
+$Comp
+L openpcharger:BAT_GND #PWR0173
+U 1 1 5E71229F
+P 2050 3550
+F 0 "#PWR0173" H 1750 3300 50  0001 C CNN
+F 1 "BAT_GND" H 2055 3377 50  0000 C CNN
+F 2 "" H 2050 3550 50  0001 C CNN
+F 3 "" H 2050 3550 50  0001 C CNN
+	1    2050 3550
+	1    0    0    -1
+$EndComp
+$Comp
+L power:GND #PWR0174
+U 1 1 5E722588
+P 3100 3550
+F 0 "#PWR0174" H 3100 3300 50  0001 C CNN
+F 1 "GND" H 3105 3377 50  0000 C CNN
+F 2 "" H 3100 3550 50  0001 C CNN
+F 3 "" H 3100 3550 50  0001 C CNN
+	1    3100 3550
+	1    0    0    -1
+$EndComp
+Wire Wire Line
+	3100 3550 3100 3450
+Wire Wire Line
+	3100 3450 2750 3450
+Connection ~ 2750 3450
 $EndSCHEMATC
