File: pcb/lipo.sch (KiCad schematic (older format))
At the start: 59 parts, among them Q3 CSD17551Q3A, Q4 CSD17551Q3A, Q5 CSD17551Q3A, Q6 CSD17551Q3A, Q7 VP0610L, U5 BQ25703ARSNT

Commit message: update
Parts:
- Q3, Q4, Q5, Q6: footprint SON65P300X350X90-9N -> Lib:SON65P300X350X90-9N
Changed lines of the file:
@@
 $Descr A4 11693 8268
 encoding utf-8
-Sheet 8 9
+Sheet 8 10
 Title ""
 Date ""
@@
 F 0 "Q6" V 7292 2650 50  0000 C CNN
 F 1 "CSD17551Q3A" V 7201 2650 50  0000 C CNN
-F 2 "SON65P300X350X90-9N" H 7150 2500 50  0001 L BNN
+F 2 "Lib:SON65P300X350X90-9N" H 7150 2500 50  0001 L BNN
 F 3 "Texas Instruments" H 7150 2500 50  0001 L BNN
 	1    7150 2500
@@
 F 0 "Q5" V 6900 2900 50  0000 L CNN
 F 1 "CSD17551Q3A" V 6800 2900 50  0000 L CNN
-F 2 "SON65P300X350X90-9N" H 6750 3050 50  0001 L BNN
+F 2 "Lib:SON65P300X350X90-9N" H 6750 3050 50  0001 L BNN
 F 3 "Texas Instruments" H 6750 3050 50  0001 L BNN
 	1    6750 3050
@@
 F 0 "Q4" V 4900 2900 50  0000 L CNN
 F 1 "CSD17551Q3A" V 4800 2900 50  0000 L CNN
-F 2 "SON65P300X350X90-9N" H 4750 3050 50  0001 L BNN
+F 2 "Lib:SON65P300X350X90-9N" H 4750 3050 50  0001 L BNN
 F 3 "Texas Instruments" H 4750 3050 50  0001 L BNN
 	1    4750 3050
@@
 F 0 "Q3" V 4500 2800 50  0000 L CNN
 F 1 "CSD17551Q3A" V 4400 2350 50  0000 L CNN
-F 2 "SON65P300X350X90-9N" H 4350 2500 50  0001 L BNN
+F 2 "Lib:SON65P300X350X90-9N" H 4350 2500 50  0001 L BNN
 F 3 "Texas Instruments" H 4350 2500 50  0001 L BNN
 	1    4350 2500
