File: pcb/mcu.sch (KiCad schematic (older format))
At the start: 7 parts, among them J1 STD14

Commit message: update
Parts:
- added C47, C48: 4.3pF, Capacitor_SMD:C_0603_1608Metric_Pad1.05x0.95mm_HandSolder, symbol Device:C_Small
- added C? (x2): 1.8pF, Capacitor_SMD:C_0603_1608Metric_Pad1.05x0.95mm_HandSolder, symbol Device:C_Small
- added C? (x7): 100nF, symbol Device:C
- added C?: 10uF, symbol Device:C
- added C? (x2): 1uF, symbol Device:C
- added C?: 4.7uF, symbol Device:C
- added D1: ESDA6V1-5SC6, Package_TO_SOT_SMD:SOT-23-6, symbol Power_Protection:ESDA6V1-5SC6
- added L? (x2): FCM1608KF-301T05, Inductor_SMD:L_0603_1608Metric_Pad1.05x0.95mm_HandSolder, symbol Device:L_Core_Ferrite
- added R? (x2): 0, symbol Device:R
- added U9: STM32G431RBT6, Package_QFP:LQFP-64_10x10mm_P0.5mm, symbol openpcharger:STM32G431RBT6
- added Y1: 32.768kHz, symbol Device:Crystal_Small
- added Y?: 8MHz, symbol Device:Crystal_Small
- R1: footprint Resistor_SMD:R_0603_1608Metric_Pad1.05x0.95mm_HandSolder -> (none)
Connections:
- net labels added: GNDA, PC14-OSC32_IN, PC15-OSC32_OUT, PF0-OSC_IN, PF1-OSC_OUT, UCPD1_CC1, UCPD1_CC2, UCPD1_DBCC1, UCPD1_DBCC2, USBPDFS_D_N, USBPDFS_D_P, USBPD_CC1, USBPD_CC2, USB_DM, USB_DP, VDDA
- wire segments 25 -> 133
Other:
- moved on the sheet: C10, C6, J1, R2, R3, R5
