File: pcb/power.sch (KiCad schematic (older format))
At the start: 7 parts, among them U1 LD3985M33R_SOT23, U4 TPS562200

Commit message: update
Parts:
- removed C1, C5: 1uF X5R, Capacitor_SMD:C_0603_1608Metric_Pad1.05x0.95mm_HandSolder, symbol Device:C
- removed C2, C4: 100nF, Capacitor_SMD:C_0603_1608Metric_Pad1.05x0.95mm_HandSolder, symbol Device:C
- removed C3: 10nF X7R, Capacitor_SMD:C_0603_1608Metric_Pad1.05x0.95mm_HandSolder, symbol Device:C
- removed U1: LD3985M33R_SOT23, Package_TO_SOT_SMD:SOT-23-5, symbol Regulator_Linear:LD3985M33R_SOT23
- removed U4: TPS562200, Package_TO_SOT_SMD:SOT-23-6, symbol Regulator_Switching:TPS562200
- added C? (x2): 68nF, 50V, symbol Device:C_Small
- added C?: 4.7uF, symbol Device:C
- added C?: 27nF, symbol Device:C
- added C?: 10pF, symbol Device:C
- added C?: 2.7nF, symbol Device:C
- added C? (x4): 1uF, symbol Device:C
- added C?: 22uF, symbol Device:C
- added C?: 33nF, symbol Device:C
- added C?: 10uF, symbol Device:C
- added C? (x2): 100nF, symbol Device:C
- added D?: LED, symbol Device:LED
- added L?: 6.8µH 4.5A, symbol Device:L_Core_Iron
- added Q? (x2): BSN20, Package_TO_SOT_SMD:SOT-23, symbol Transistor_FET:BSN20
- added R?: 200K, symbol Device:R
- added R?: 49.9K, symbol Device:R
- added R?: 4.22K, symbol Device:R
- added R?: 1.05M, symbol Device:R
- added R?: 787K, symbol Device:R
- added R?: 64.9K, symbol Device:R
- added R?: 180K, symbol Device:R
- added R? (x2): 10K, symbol Device:R
- added R?: 59K, symbol Device:R
- added R?: 0, symbol Device:R
- added R?: 330, symbol Device:R
- added U?: LTC3114EFE-1, Lib:SOP65P640X110-17N, symbol LTC3114EFE-1_TRPBF:LTC3114EFE-1#TRPBF
- added U?: LD39050PU33R, Lib:SON95P300X300X100-7N, symbol LD39050PU33R:LD39050PU33R
Connections:
- net GND: now also C?.2, C?.2, C?.2, C?.2, C?.2, C?.2, C?.2, C?.2, C?.2, C?.2, C?.2, C?.2, D?.1 (K), Q?.2 (S), Q?.2 (S), R?.2, R?.2, R?.2, R?.2, R?.2, U?.1 (PGND), U?.16 (MODE), U?.17 (PGND), U?.2 (GND), U?.7 (GND), U?.8 (GND)
- new net: C?.2, U?.12 (BST2)
- new net: C?.2, U?.13 (BST1)
- new net: C?.1, R?.2
- new net: Q?.3 (D), R?.2 (x2)
- new net: C?.1, C?.1, R?.1, R?.2, U?.4 (VOUT)
- new net: D?.2 (A), R?.2
- new net FB: C?.2, R?.1, R?.2, U?.7 (FB)
- new net LDO_PLDO: C?.1, U?.11 (PLDO), U?.9 (LDO)
- new net PROG: C?.1, R?.1, R?.1, R?.1, U?.5 (PROG)
- new net RUN: R?.1, R?.2, U?.4 (RUN)
- new net SW1: C?.1, L?.1, U?.15 (SW1)
- new net SW2: C?.1, L?.2, U?.2 (SW2)
- new net USBPD_1A_PROTECT: Q?.1 (G), R?.1
- new net USBPD_550mA_PROTECT: Q?.1 (G), R?.1
- new net VBUS: C?.1, C?.1, R?.1, U?.10 (VIN), U?.14 (PVIN)
- new net VBUS_5V: C?.1, C?.1, C?.1, C?.1, C?.1, R?.1, U?.1 (EN), U?.3 (PVOUT), U?.6 (VIN)
- new net VC: C?.1, R?.1, U?.6 (VC)
- new net VDD: R?.1
- no-connect marks 0 -> 1
Other:
- note added: "Iout=25000/R"
- note added: "USB PD 5V Converter"
