File: pcb/usb.sch (KiCad schematic (older format))
At the start: 25 parts, among them J2 USB_C_Receptacle, Q1 STL6P3LLH6, Q2 STL9P3LLH6, U2 USBLC6-2SC6, U6 LD39050PU33R, U7 LTC3114EFE-1#TRPBF

Commit message: update
Parts:
- removed C11, C12: 68nF, 50V, symbol Device:C_Small
- removed C13: 27nF, symbol Device:C
- removed C14: 10pF, symbol Device:C
- removed C15: 4.7uF, symbol Device:C
- removed C16: 2.7nF, symbol Device:C
- removed C17, C? (x2): 1uF, symbol Device:C
- removed C18: 22uF, symbol Device:C
- removed C? (x2): 100nF, symbol Device:C
- removed D?: LED, symbol Device:LED
- removed L1: 6.8µH 4.5A, symbol Device:L_Core_Iron
- removed Q2: STL9P3LLH6, TRANS_STL9P3LLH6, symbol STL9P3LLH6:STL9P3LLH6
- removed R6: 4.22K, symbol Device:R
- removed R7: 200K, symbol Device:R
- removed R8: 49.9K, symbol Device:R
- removed R?: 330, symbol Device:R
- removed R?: 0, symbol Device:R
- removed U6: LD39050PU33R, SON95P300X300X100-7N, symbol LD39050PU33R:LD39050PU33R
- removed U7: LTC3114EFE-1#TRPBF, SOP65P640X110-17N, symbol LTC3114EFE-1_TRPBF:LTC3114EFE-1#TRPBF
- added C49: 100nF, symbol Device:C
- added C? (x2): 390pF, Capacitor_SMD:C_0603_1608Metric_Pad1.05x0.95mm_HandSolder, symbol Device:C
- added D?: SP0502BAHT, Package_TO_SOT_SMD:SOT-23, symbol Power_Protection:SP0502BAHT
- added D?: 5KPxxA, Diode_THT:D_P600_R-6_P20.00mm_Horizontal, symbol Diode:5KPxxA
Connections:
- net GND: now also C49.2, C?.2, C?.2, D?.2 (A2), D?.3 (A)
- net VBUS: now also C49.1, D?.1 (A1)
- net USBPD_CC1: now reaches J2.A5 (CC1)
- net USBPD_CC1: now also C?.1, D?.1 (K)
- net USBPD_CC2: now reaches J2.B5 (CC2)
- net USBPD_CC2: now also C?.1, D?.2 (K)
- no-connect marks 11 -> 10
Other:
- note added: "Change TVS"
- moved on the sheet: Q1
